File: kicad/metal detector test/metal detector test.kicad_pcb (KiCad board)
At the start: 2 copper layers, 72.6 x 125 mm, 110 parts, among them J1 3.5mm audio jack TRS, Q1 PNP, Q2 NPN, SW1 SW_SPST, SW10 SW_SPST, SW2 SW_SPST, SW3 SW_SPST, SW4 SW_SPST, SW5 SW_SPST, SW6 SW_SPST, SW7 SW_SPST, SW8 SW_SPST, SW9 SW_SPST, U1 op amp (higher voltage), U10 3.3v lin reg, U11 lp filter, U12 op amp (lower voltage), U2 nucleo-32 uC module, U3 9v lin reg, U4 5v lin reg, U5 3.3v lin reg, U6 audio amp, U7 lp filter, U8 switch debounce, U9 5v lin reg

Commit message: small changes
Parts:
- moved C13 143.9 mm to (76.2, 112.3), turned to -90 degrees
- moved U8 139.9 mm to (70.6, 104.1)
- moved SW6 113.5 mm to (94.7, 102.9)
- moved SW7 113.5 mm to (87.1, 102.9)
- moved SW8 113.5 mm to (87.1, 94.1)
- moved SW9 113.5 mm to (79.5, 94.1)
- moved SW10 113.5 mm to (71.9, 94.1)
- moved SW2 113.5 mm to (117.6, 94.1)
- moved SW3 113.5 mm to (110.0, 94.1)
- moved SW4 113.5 mm to (102.4, 94.1)
- moved SW5 113.5 mm to (102.4, 102.9)
Changed lines of the file:
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@@
   )
   (footprint "allen footprints:SW_SPST_PTS647" placed (layer "B.Cu")
-    (at 200.406 96.598 180)
+    (at 87.122 102.948 180)
     (descr "C&K Components SPST SMD PTS647 Series 4.5mm Tact Switch")
     (tags "SPST Button Switch")
@@
   )
   (footprint "allen footprints:SW_SPST_PTS647" placed (layer "B.Cu")
-    (at 200.406 87.708 180)
+    (at 87.122 94.058 180)
     (descr "C&K Components SPST SMD PTS647 Series 4.5mm Tact Switch")
     (tags "SPST Button Switch")
@@
   )
   (footprint "Capacitor_SMD:C_0805_2012Metric_Pad1.18x1.45mm_HandSolder" (layer "B.Cu")
-    (at 216.027 78.31 90)
+    (at 76.2 112.268 -90)
     (descr "Capacitor SMD 0805 (2012 Metric), square (rectangular) end terminal, IPC_7351 nominal with elongated pad for handsoldering. (Body size source: IPC-SM-782 page 76, https://www.pcb-3d.com/wordpress/wp-content/uploads/ipc-sm-782a_amendment_1_and_2.pdf, https://docs.google.com/spreadsheets/d/1BsfQQcO9C6DZCsRaXUlFlo91Tg2WpOkGARC1WS5S8t0/edit?usp=sharing), generated with kicad-footprint-generator")
     (tags "capacitor handsolder")
@@
     (fp_line (start 1 0.625) (end 1 -0.625)
       (stroke (width 0.1) (type solid)) (layer "B.Fab"))
-    (pad "1" smd roundrect (at -1.0375 0 90) (size 1.175 1.45) (layers "B.Cu" "B.Paste" "B.Mask") (roundrect_rratio 0.212766)
+    (pad "1" smd roundrect (at -1.0375 0 270) (size 1.175 1.45) (layers "B.Cu" "B.Paste" "B.Mask") (roundrect_rratio 0.212766)
       (net 19 "+3.3V_uC") (pintype "passive"))
-    (pad "2" smd roundrect (at 1.0375 0 90) (size 1.175 1.45) (layers "B.Cu" "B.Paste" "B.Mask") (roundrect_rratio 0.212766)
+    (pad "2" smd roundrect (at 1.0375 0 270) (size 1.175 1.45) (layers "B.Cu" "B.Paste" "B.Mask") (roundrect_rratio 0.212766)
       (net 2 "GNDA") (pintype "passive"))
     (model "${KICAD6_3DMODEL_DIR}/Capacitor_SMD.3dshapes/C_0805_2012Metric.wrl"
@@
   )
   (footprint "allen footprints:SW_SPST_PTS647" placed (layer "B.Cu")
-    (at 208.026 96.598 180)
+    (at 94.742 102.948 180)
     (descr "C&K Components SPST SMD PTS647 Series 4.5mm Tact Switch")
     (tags "SPST Button Switch")
@@
   )
   (footprint "allen footprints:SW_SPST_PTS647" placed (layer "B.Cu")
-    (at 192.786 87.708 180)
+    (at 79.502 94.058 180)
     (descr "C&K Components SPST SMD PTS647 Series 4.5mm Tact Switch")
     (tags "SPST Button Switch")
@@
   )
   (footprint "allen footprints:SW_SPST_PTS647" placed (layer "B.Cu")
-    (at 215.646 87.708 180)
+    (at 102.362 94.058 180)
     (descr "C&K Components SPST SMD PTS647 Series 4.5mm Tact Switch")
     (tags "SPST Button Switch")
@@
   )
   (footprint "Package_SO:SOIC-20W_7.5x12.8mm_P1.27mm" placed (layer "B.Cu")
-    (at 208.026 77.978 90)
+    (at 70.612 104.14 90)
     (descr "SOIC, 20 Pin (JEDEC MS-013AC, https://www.analog.com/media/en/package-pcb-resources/package/233848rw_20.pdf), generated with kicad-footprint-generator ipc_gullwing_generator.py")
     (tags "SOIC SO")
@@
   )
   (footprint "allen footprints:SW_SPST_PTS647" placed (layer "B.Cu")
-    (at 230.886 87.708 180)
+    (at 117.602 94.058 180)
     (descr "C&K Components SPST SMD PTS647 Series 4.5mm Tact Switch")
     (tags "SPST Button Switch")
@@
   )
   (footprint "allen footprints:SW_SPST_PTS647" placed (layer "B.Cu")
-    (at 185.166 87.708 180)
+    (at 71.882 94.058 180)
     (descr "C&K Components SPST SMD PTS647 Series 4.5mm Tact Switch")
     (tags "SPST Button Switch")
@@
   )
   (footprint "allen footprints:SW_SPST_PTS647" placed (layer "B.Cu")
-    (at 215.646 96.598 180)
+    (at 102.362 102.948 180)
     (descr "C&K Components SPST SMD PTS647 Series 4.5mm Tact Switch")
     (tags "SPST Button Switch")
@@
   )
   (footprint "allen footprints:SW_SPST_PTS647" placed (layer "B.Cu")
-    (at 223.266 87.708 180)
+    (at 109.982 94.058 180)
     (descr "C&K Components SPST SMD PTS647 Series 4.5mm Tact Switch")
     (tags "SPST Button Switch")
